File: kicad/munlite.kicad_pcb (KiCad board)
At the start: 2 copper layers, 45.7 x 24.9 mm, 21 parts, among them J1 Conn_Pover, J2 Conn_Pir, J3 Conn_Prog, J4 Conn_Opto, J5 Conn_Led, SW1 SW_Push, U1 STM32L031F6Px, U2 AP2112K-3.3, U3 CN5711

Commit message: to update
Routing:
- net +4V: track 27.6 -> 28.3 mm
Changed lines of the file:
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@@
       (dxfimperialunits true)
       (dxfusepcbnewfont true)
-      (psnegative false)
+      (psnegative true)
       (psa4output false)
       (plotreference false)
@@
       (subtractmaskfromsilk false)
       (outputformat 5)
-      (mirror true)
+      (mirror false)
       (drillshape 2)
       (scaleselection 1)
@@
     (fp_line (start -1.6 -0.8) (end 1.6 -0.8) (layer "F.Fab") (width 0.1))
     (fp_line (start -1.6 0.8) (end -1.6 -0.8) (layer "F.Fab") (width 0.1))
-    (pad "1" smd roundrect (at -1.4625 0 90) (size 1.125 1.75) (layers "F.Cu" "F.Paste" "F.Mask") (roundrect_rratio 0.222222)
+    (pad "1" smd roundrect (at -1.4625 0 90) (size 1.125 1.75) (layers "F.Cu" "F.Paste" "F.Mask") (roundrect_rratio 0.2222222222)
       (net 3 "GND"))
-    (pad "2" smd roundrect (at 1.4625 0 90) (size 1.125 1.75) (layers "F.Cu" "F.Paste" "F.Mask") (roundrect_rratio 0.222222)
+    (pad "2" smd roundrect (at 1.4625 0 90) (size 1.125 1.75) (layers "F.Cu" "F.Paste" "F.Mask") (roundrect_rratio 0.2222222222)
       (net 3 "GND"))
     (model "${KICAD6_3DMODEL_DIR}/Resistor_SMD.3dshapes/R_1206_3216Metric.wrl"
@@
   (segment (start 64.582 42.672) (end 62.992 44.262) (width 0.5) (layer "F.Cu") (net 1))
   (segment (start 44.831 41.275) (end 44.308 40.752) (width 0.5) (layer "F.Cu") (net 1))
-  (segment (start 67.437 52.451) (end 67.437 54.737) (width 1) (layer "F.Cu") (net 2))
   (segment (start 78.17 55.626) (end 78.17 55.688) (width 0.5) (layer "F.Cu") (net 2))
-  (segment (start 69.215 56.515) (end 77.343 56.515) (width 1) (layer "F.Cu") (net 2))
+  (segment (start 67.437 55.245) (end 69.215 57.023) (width 1) (layer "F.Cu") (net 2))
   (segment (start 66.179 46.421) (end 68.0775 46.421) (width 0.3) (layer "F.Cu") (net 2))
+  (segment (start 76.835 57.023) (end 77.343 56.515) (width 1) (layer "F.Cu") (net 2))
   (segment (start 78.17 55.688) (end 77.343 56.515) (width 0.5) (layer "F.Cu") (net 2))
-  (segment (start 67.437 54.737) (end 69.215 56.515) (width 1) (layer "F.Cu") (net 2))
+  (segment (start 67.437 52.451) (end 67.437 55.245) (width 1) (layer "F.Cu") (net 2))
   (segment (start 65.405 50.419) (end 65.405 47.195) (width 1) (layer "F.Cu") (net 2))
   (segment (start 66.785 48.321) (end 68.0775 48.321) (width 0.3) (layer "F.Cu") (net 2))
@@
   (segment (start 65.532 47.068) (end 66.785 48.321) (width 0.3) (layer "F.Cu") (net 2))
   (segment (start 65.405 47.195) (end 65.532 47.068) (width 1) (layer "F.Cu") (net 2))
+  (segment (start 69.215 57.023) (end 76.835 57.023) (width 1) (layer "F.Cu") (net 2))
   (segment (start 41.402 39.243) (end 41.402 49.272) (width 0.5) (layer "F.Cu") (net 3))
   (segment (start 72.517 49.53) (end 72.517 47.625) (width 1) (layer "F.Cu") (net 3))
